File: Hardware/Schemas/Bachelorproef V1/Bachelorproef V1.kicad_sch (KiCad schematic)
At the start: 42 parts, among them J1 EA W096016-XALW, P1 USB_C_Plug, SW1 Reset, U1 ATMEGA328P-AU, U2 BME680, U3 FT232RL, U4 PI6ULS5V9306

Commit message: Add files via upload
Parts:
- U4: value PI6ULS5V9306 -> PCA9306DCUR
Changed lines of the file:
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@@
     (in_bom yes) (on_board yes) (fields_autoplaced)
     (property "Reference" "U4" (id 0) (at 137.16 99.06 0))
-    (property "Value" "PI6ULS5V9306" (id 1) (at 137.16 101.6 0))
+    (property "Value" "PCA9306DCUR" (id 1) (at 137.16 101.6 0))
     (property "Footprint" "TCA9517ADGKR:TCA9517ADGKR" (id 2) (at 209.55 41.91 0)
       (effects (font (size 1.27 1.27)) (justify left) hide)
@@
     )
     (path "/218d8b52-6b66-40f6-a5de-c0bd454da8da"
-      (reference "U4") (unit 1) (value "PI6ULS5V9306") (footprint "TCA9517ADGKR:TCA9517ADGKR")
+      (reference "U4") (unit 1) (value "PCA9306DCUR") (footprint "TCA9517ADGKR:TCA9517ADGKR")
     )
     (path "/9ac4cf03-7929-44dd-9f74-8225f7549cd2"
