File: Hardware/Schemas/Bachelorproef V2/Bachelorproef V2.kicad_pcb (KiCad board)
At the start: 2 copper layers, 48 x 15 mm, 40 parts, among them IC2 TCA9517ADGKR, J1 EA W096016-XALW, P1 USB_C_Plug, SW1 Reset, U2 MCP1700T-3302E/TT, U3 BME680

Commit message: Add files via upload
Parts:
- removed R13: 10kΩ, Resistor_SMD:R_0603_1608Metric_Pad0.98x0.95mm_HandSolder
- added ?: , , F.Cu at (160.7, 97.9)
- added ?: , , F.Cu at (160.7, 85.9)
- added ?: , , F.Cu at (115.7, 97.9)
- added ?: , , F.Cu at (115.7, 85.9)
- added ATmega32U4: ATMEGA32U4-AU, ATMEGA32U4-AU:ATMEGA32U4-AU, B.Cu at (124.9, 91.9)
- C1, C10, C11, C12, C14, C15, C3, C4, C5, C6, C7, C8, C9, IC2, J1, R1, R10, R11, R12, R5, R6, R9, U2, U3, XTAL1: moved to B.Cu
- C13: value 1µF -> 100nF; moved to B.Cu
- P1: footprint USB4155-03-C:USB4155-03-C -> CX60-24S-UNIT:CX60-24S-UNIT
- R14: value 390kΩ -> 910kΩ; moved to B.Cu
- R3: value 150Ω -> 1.5kΩ
- R7, R8: value 120Ω -> 1.5kΩ
- moved C4 55.6 mm to (115.8, 89.3), turned to -90 degrees
- moved C5 47.9 mm to (115.8, 92.5), turned to -90 degrees
- moved R3 47.6 mm to (125.7, 85.7), turned to 180 degrees
- moved F1 45.4 mm to (119.2, 89.2), turned to 180 degrees
- moved R4 45.4 mm to (122.2, 85.7)
- moved R2 45.3 mm to (144.9, 85.6), turned to 180 degrees
- moved D1 44.8 mm to (129.2, 85.7), turned to 180 degrees
- moved C3 41.3 mm to (134.3, 91.9)
- moved C6 40.7 mm to (132.9, 94.3), turned to 90 degrees
- moved R6 40.4 mm to (133.8, 90.0)
- moved C1 38.6 mm to (147.7, 88.0)
- moved C14 38.3 mm to (147.6, 91.6), turned to 180 degrees
- moved R14 38.3 mm to (156.7, 85.5)
- moved C2 38.1 mm to (126.8, 97.8)
- moved C12 38.0 mm to (152.7, 85.5)
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Connections:
- C12 pad 2: Net-(C12-Pad2) -> GND
- C13 pad 1: +3V3 -> Net-(C13-Pad1)
- C13 pad 2: Net-(C13-Pad2) -> GND
- C14 pad 1: Net-(C14-Pad1) -> Net-(C13-Pad1)
- J1 pad 13: Net-(C14-Pad1) -> Net-(C13-Pad1)
- J1 pad 5: Net-(C13-Pad2) -> +3V3
- J1 pad 8: Net-(C12-Pad2) -> +3V3
- J1 pad 9: Net-(J1-Pad9) -> RES
Routing:
- net GND: track 0.00 -> 215.5 mm, vias 0 -> 10
- net +5V: track 0.00 -> 117.6 mm, vias 0 -> 13
- net SCL 5V: track 0.00 -> 51.5 mm, vias 0 -> 3
- net +3V3: track 0.00 -> 50.8 mm, vias 0 -> 3
- net Net-(F1-Pad1): track 0.00 -> 44.7 mm, vias 0 -> 2
- net SDA 5V: track 0.00 -> 41.4 mm, vias 0 -> 5
- net TXLED: track 0.00 -> 22.4 mm, vias 0 -> 1
- net D-: track 0.00 -> 21.3 mm, vias 0 -> 1
- net RESET: track 0.00 -> 19.1 mm, vias 0 -> 3
- net D+: track 0.00 -> 18.4 mm, vias 0 -> 1
- net Net-(P1-PadA5): track 0.00 -> 17.5 mm, vias 0 -> 2
- net SDA 3V3: track 0.00 -> 16.9 mm, vias 0 -> 3
- net XTAL2: track 0.00 -> 16.7 mm
- net RXLED: track 0.00 -> 16.3 mm, vias 0 -> 1
- net SCL 3V3: track 0.00 -> 15.9 mm
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Other:
- board size 48 x 15 mm -> 48 x 18.9 mm
- board text added: "OLED DISPLAY"
