File: Hardware/Schemas/Bachelorproef V2/Bachelorproef V2.kicad_pcb (KiCad board)
At the start: 2 copper layers, 48 x 18.9 mm, 44 parts, among them IC2 TCA9517ADGKR, J1 EA W096016-XALW, P1 USB_C_Plug, SW1 Reset, U2 MCP1700T-3302E/TT, U3 BME680

Commit message: Add files via upload
Parts:
- added R15: 5.1kΩ, Resistor_SMD:R_0603_1608Metric_Pad0.98x0.95mm_HandSolder, F.Cu at (149.5, 85.5)
- added R16: 10kΩ, Resistor_SMD:R_0603_1608Metric_Pad0.98x0.95mm_HandSolder, F.Cu at (153.0, 85.5)
Connections:
- ATmega32U4 pad 41: unconnected-(U1-Pad41) -> RES#
- J1 pad 9: RES -> Net-(J1-Pad9)
Routing:
- net RES#: track 0.00 -> 28.5 mm, vias 0 -> 1
- net Net-(J1-Pad9): track 0.00 -> 10.1 mm, vias 0 -> 1
- net GND: track 215.5 -> 220.2 mm, vias 10 -> 11
- net +3V3: track 50.8 -> 51.7 mm
