File: Hardware/Schemas/Bachelorproef V2/Bachelorproef V2.kicad_sch (KiCad schematic)
At the start: 41 parts, among them IC2 TCA9517ADGKR, J1 EA W096016-XALW, P1 USB_C_Plug, SW1 Reset, U1 ATMEGA32U4-AU, U2 MCP1700T-3302E/TT, U3 BME680

Commit message: Add files via upload
Parts:
- R14: value 390kΩ -> 910kΩ
- R7, R8: value 120Ω -> 150Ω
Changed lines of the file:
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@@
       (effects (font (size 1.27 1.27)) (justify left))
     )
-    (property "Value" "120Ω" (id 1) (at 83.82 82.55 0)
+    (property "Value" "150Ω" (id 1) (at 83.82 82.55 0)
       (effects (font (size 1.27 1.27)) (justify left))
     )
@@
       (effects (font (size 1.27 1.27)) (justify left))
     )
-    (property "Value" "390kΩ" (id 1) (at 195.58 148.59 0)
+    (property "Value" "910kΩ" (id 1) (at 195.58 148.59 0)
       (effects (font (size 1.27 1.27)) (justify left))
     )
@@
       (effects (font (size 1.27 1.27)) (justify left))
     )
-    (property "Value" "120Ω" (id 1) (at 96.52 82.55 0)
+    (property "Value" "150Ω" (id 1) (at 96.52 82.55 0)
       (effects (font (size 1.27 1.27)) (justify left))
     )
@@
     )
     (path "/72919f65-1b8c-4d67-acfd-9e30bd2605d1"
-      (reference "R7") (unit 1) (value "120Ω") (footprint "Resistor_SMD:R_0603_1608Metric_Pad0.98x0.95mm_HandSolder")
+      (reference "R7") (unit 1) (value "150Ω") (footprint "Resistor_SMD:R_0603_1608Metric_Pad0.98x0.95mm_HandSolder")
     )
     (path "/fc08deda-f04f-47a5-a6fd-1fbcb9951de6"
-      (reference "R8") (unit 1) (value "120Ω") (footprint "Resistor_SMD:R_0603_1608Metric_Pad0.98x0.95mm_HandSolder")
+      (reference "R8") (unit 1) (value "150Ω") (footprint "Resistor_SMD:R_0603_1608Metric_Pad0.98x0.95mm_HandSolder")
     )
     (path "/3a543739-361f-437c-a325-3a8e29f1f40f"
@@
     )
     (path "/872b1738-1647-4c8e-8f4a-96832859fff8"
-      (reference "R14") (unit 1) (value "390kΩ") (footprint "Resistor_SMD:R_0603_1608Metric_Pad0.98x0.95mm_HandSolder")
+      (reference "R14") (unit 1) (value "910kΩ") (footprint "Resistor_SMD:R_0603_1608Metric_Pad0.98x0.95mm_HandSolder")
     )
     (path "/0a0fbdf1-3683-4392-9ad2-e725a5eb7726"

Commit message: Add files via upload
Parts:
- removed R13: 10kΩ, Resistor_SMD:R_0603_1608Metric_Pad0.98x0.95mm_HandSolder, symbol Device:R
- C13: value 1µF -> 100nF
- R3, R7, R8: value 150Ω -> 680Ω
Connections:
- net +3V3: now also J1.5 (VBAT), J1.8 (VDD); no longer C13.1
- net GND: now also C12.2, C13.2
- net at C14.1, J1.13 (VCOMH): now also C13.1
- net RES: now reaches J1.9 (RES#)
Other:
- moved on the sheet: C12, C13, C14, C15, R14

Commit message: Add files via upload
Parts:
- P1: footprint USB4155-03-C:USB4155-03-C -> CX60-24S-UNIT:CX60-24S-UNIT
- R3, R7, R8: value 680Ω -> 1.5kΩ
- U1: footprint (none) -> ATMEGA32U4-AU:ATMEGA32U4-AU
Other:
- moved on the sheet: C1, C2, C8, C9, D1, F1, P1, R1, R2, R3, U2

Commit message: Add files via upload
Parts:
- added R15: 5.1kΩ, Resistor_SMD:R_0603_1608Metric_Pad0.98x0.95mm_HandSolder, symbol Device:R
- added R16: 10kΩ, Resistor_SMD:R_0603_1608Metric_Pad0.98x0.95mm_HandSolder, symbol Device:R
- renumbered U1 to ATmega32U4
Connections:
- net GND: now also R16.2
- net RES#: now reaches ATmega32U4.41 (PF0)
- net RES#: now also R15.1
- net RES: no longer names the net of J1.9 (RES#)
- net RES: now also R15.2, R16.1
Other:
- moved on the sheet: IC2, R10, R11, R12, R9
